Commit message: Added physical inertial properties to all links

File: my_robot.urdf (robot description, URDF)
Before this commit: robot my_robot, 4 links, 3 joints
Links:
- removed link wheel
- added link wheel_left, mass 0.5; collision cylinder length=0.05 radius=0.1; visual cylinder length=0.05 radius=0.1
- link base_link: mass None -> 5.0; geometry collision box size=0.5 0.3 0.1; visual box size=0.5 0.3 0.1
- link caster_wheel: mass None -> 0.1
- link wheel_right: mass None -> 0.5; geometry collision cylinder length=0.05 radius=0.1; visual cylinder length=0.05 radius=0.1
Joints:
- joint base_to_wheel: child wheel -> wheel_left

Commit message: Fixed caster wheel ground penetration by using sphere collision

File: my_robot.urdf (robot description, URDF)
Before this commit: robot my_robot, 4 links, 3 joints
Links:
- link caster_wheel: geometry collision sphere radius=0.05; visual sphere radius=0.05

Commit message: Added LiDAR visual link and joint

File: my_robot.urdf (robot description, URDF)
Before this commit: robot my_robot, 4 links, 3 joints
Links:
- added link laser_frame, mass 0.1; collision cylinder length=0.04 radius=0.05; visual cylinder length=0.04 radius=0.05
Joints:
- added joint laser_joint: type fixed, parent base_link, child laser_frame, origin xyz=0 0 0.17 rpy=0 0 0

Commit message: LiDAR is fully functional with range data and scan topic

File: my_robot.urdf (robot description, URDF)
Before this commit: robot my_robot, 5 links, 4 joints
Joints:
- joint laser_joint: origin xyz=0 0 0.17 rpy=0 0 0 -> xyz=0 0 0.25 rpy=0 0 0
